File: pizero_grbl_hat.sch (KiCad schematic (older format))
At the start: 16 parts, among them J1 GPIO_CONNECTOR

Commit message: finish schematics, start assigning packages
Parts:
- added A1: X-axis, Module:Pololu_Breakout-16_15.2x20.3mm, symbol Driver_Motor:Pololu_Breakout_DRV8825
- added A2: Y-axis, Module:Pololu_Breakout-16_15.2x20.3mm, symbol Driver_Motor:Pololu_Breakout_DRV8825
- added C1: 100n, Capacitor_SMD:C_0805_2012Metric, symbol Device:C
- added C8: 100u, symbol Device:CP
- added J3: LIMIT_X, symbol Connector_Generic:Conn_01x02
- added J4: LIMIT_Y, symbol Connector_Generic:Conn_01x02
- added J5: VMOT, symbol Connector_Generic:Conn_01x02
- added J6: MOTOR_X, symbol Connector_Generic:Conn_01x04
- added J7: MOTOR_Y, symbol Connector_Generic:Conn_01x04
- added TP1, TP2, TP3, TP4, TP5, TP6: TestPoint_2Pole, symbol Connector:TestPoint_2Pole
- C2, C3, C4, C5, C6, C7: renamed from C?; footprint (none) -> Capacitor_SMD:C_0805_2012Metric
- R1, R2: renamed from R?; footprint (none) -> Resistor_SMD:R_0805_2012Metric
- gave numbers to parts that had none: 3
Connections:
- net GPIO14_TXD0 is gone; now on net RXD: J1.8 (Pin_8)
- net GPIO15_RXD0 is gone; now on net TXD: J1.10 (Pin_10)
- net +3V3: now also A1.13 (~RST), A1.14 (~SLP), A2.13 (~RST), A2.14 (~SLP), C1.1, TP1.1, TP2.1, TP3.1, TP4.1, TP5.1, TP6.1
- net DIRX: now also A1.16 (DIR)
- net DIRY: now also A2.16 (DIR)
- net EN: now also A1.9 (~EN), A2.9 (~EN)
- net GND: now also A1.1 (GND), A1.7 (GND), A2.1 (GND), A2.7 (GND), C1.2, C8.2, J3.2 (Pin_2), J4.2 (Pin_2), J5.2 (Pin_2)
- net LIMITX: now also J3.1 (Pin_1)
- net LIMITY: now also J4.1 (Pin_1)
- net STEPX: now also A1.15 (STEP)
- net STEPY: now also A2.15 (STEP)
- new net: A1.10 (M0), TP1.2
- new net: A1.11 (M1), TP2.2
- new net: A1.12 (M2), TP3.2
- new net: A1.3 (A2), J6.2 (Pin_2)
- new net: A1.4 (A1), J6.1 (Pin_1)
- new net: A1.5 (B1), J6.3 (Pin_3)
- new net: A1.6 (B2), J6.4 (Pin_4)
- new net: A1.8 (VMOT), A2.8 (VMOT), C8.1, J5.1 (Pin_1)
- new net: A2.10 (M0), TP4.2
- new net: A2.11 (M1), TP5.2
- new net: A2.12 (M2), TP6.2
- new net: A2.3 (A2), J7.2 (Pin_2)
- new net: A2.4 (A1), J7.1 (Pin_1)
- new net: A2.5 (B1), J7.3 (Pin_3)
- new net: A2.6 (B2), J7.4 (Pin_4)
- no-connect marks 37 -> 38
Other:
- note added: "Limit switches: Normally open, pull to GND to engage"
- moved on the sheet: C2, C4, C5, J2, R1, R2, U1, Y1

Commit message: layout mostly done
Parts:
- C8: footprint (none) -> Capacitor_SMD:CP_Elec_6.3x7.7
- J2: footprint (none) -> Connector_PinHeader_2.54mm:PinHeader_2x03_P2.54mm_Vertical
- J3, J4, J5: footprint (none) -> Connector_JST:JST_PH_B2B-PH-K_1x02_P2.00mm_Vertical
- J6, J7: footprint (none) -> Connector_JST:JST_PH_B4B-PH-K_1x04_P2.00mm_Vertical
- TP1, TP2, TP3, TP4, TP5, TP6: footprint (none) -> TestPoint:TestPoint_2Pads_Pitch2.54mm_Drill0.8mm
- Y1: footprint (none) -> Crystal:Crystal_SMD_2012-2Pin_2.0x1.2mm
Changed lines of the file:
@@
 F 0 "Y1" V 3604 2331 50  0000 L CNN
 F 1 "16MHz" V 3695 2331 50  0000 L CNN
-F 2 "" H 3650 2200 50  0001 C CNN
+F 2 "Crystal:Crystal_SMD_2012-2Pin_2.0x1.2mm" H 3650 2200 50  0001 C CNN
 F 3 "~" H 3650 2200 50  0001 C CNN
 	1    3650 2200
@@
 F 0 "J2" H 4200 1367 50  0000 C CNN
 F 1 "ISP" H 4200 1276 50  0000 C CNN
-F 2 "" H 4150 1050 50  0001 C CNN
+F 2 "Connector_PinHeader_2.54mm:PinHeader_2x03_P2.54mm_Vertical" H 4150 1050 50  0001 C CNN
 F 3 "~" H 4150 1050 50  0001 C CNN
 	1    4150 1050
@@
 F 0 "J7" H 10330 2542 50  0000 L CNN
 F 1 "MOTOR_Y" H 10330 2451 50  0000 L CNN
-F 2 "" H 10250 2550 50  0001 C CNN
+F 2 "Connector_JST:JST_PH_B4B-PH-K_1x04_P2.00mm_Vertical" H 10250 2550 50  0001 C CNN
 F 3 "~" H 10250 2550 50  0001 C CNN
 	1    10250 2550
@@
 F 0 "J5" H 6118 1517 50  0000 C CNN
 F 1 "VMOT" H 6118 1426 50  0000 C CNN
-F 2 "" H 6200 1300 50  0001 C CNN
+F 2 "Connector_JST:JST_PH_B2B-PH-K_1x02_P2.00mm_Vertical" H 6200 1300 50  0001 C CNN
 F 3 "~" H 6200 1300 50  0001 C CNN
 	1    6200 1300
@@
 F 0 "C8" H 6768 1496 50  0000 L CNN
 F 1 "100u" H 6768 1405 50  0000 L CNN
-F 2 "" H 6688 1300 50  0001 C CNN
+F 2 "Capacitor_SMD:CP_Elec_6.3x7.7" H 6688 1300 50  0001 C CNN
 F 3 "~" H 6650 1450 50  0001 C CNN
 	1    6650 1450
@@
 F 0 "TP1" H 6000 3153 50  0000 C CNN
 F 1 "TestPoint_2Pole" H 6000 3154 50  0001 C CNN
-F 2 "" H 6000 3050 50  0001 C CNN
+F 2 "TestPoint:TestPoint_2Pads_Pitch2.54mm_Drill0.8mm" H 6000 3050 50  0001 C CNN
 F 3 "~" H 6000 3050 50  0001 C CNN
 	1    6000 3050
@@
 F 0 "TP2" H 6000 3353 50  0000 C CNN
 F 1 "TestPoint_2Pole" H 6000 3354 50  0001 C CNN
-F 2 "" H 6000 3250 50  0001 C CNN
+F 2 "TestPoint:TestPoint_2Pads_Pitch2.54mm_Drill0.8mm" H 6000 3250 50  0001 C CNN
 F 3 "~" H 6000 3250 50  0001 C CNN
 	1    6000 3250
@@
 F 0 "TP3" H 6000 3553 50  0000 C CNN
 F 1 "TestPoint_2Pole" H 6000 3554 50  0001 C CNN
-F 2 "" H 6000 3450 50  0001 C CNN
+F 2 "TestPoint:TestPoint_2Pads_Pitch2.54mm_Drill0.8mm" H 6000 3450 50  0001 C CNN
 F 3 "~" H 6000 3450 50  0001 C CNN
 	1    6000 3450
@@
 F 0 "TP4" H 8550 3153 50  0000 C CNN
 F 1 "TestPoint_2Pole" H 8550 3154 50  0001 C CNN
-F 2 "" H 8550 3050 50  0001 C CNN
+F 2 "TestPoint:TestPoint_2Pads_Pitch2.54mm_Drill0.8mm" H 8550 3050 50  0001 C CNN
 F 3 "~" H 8550 3050 50  0001 C CNN
 	1    8550 3050
@@
 F 0 "TP5" H 8550 3353 50  0000 C CNN
 F 1 "TestPoint_2Pole" H 8550 3354 50  0001 C CNN
-F 2 "" H 8550 3250 50  0001 C CNN
+F 2 "TestPoint:TestPoint_2Pads_Pitch2.54mm_Drill0.8mm" H 8550 3250 50  0001 C CNN
 F 3 "~" H 8550 3250 50  0001 C CNN
 	1    8550 3250
@@
 F 0 "TP6" H 8550 3553 50  0000 C CNN
 F 1 "TestPoint_2Pole" H 8550 3554 50  0001 C CNN
-F 2 "" H 8550 3450 50  0001 C CNN
+F 2 "TestPoint:TestPoint_2Pads_Pitch2.54mm_Drill0.8mm" H 8550 3450 50  0001 C CNN
 F 3 "~" H 8550 3450 50  0001 C CNN
 	1    8550 3450
@@
 F 0 "J3" H 4480 4192 50  0000 L CNN
 F 1 "LIMIT_X" H 4480 4101 50  0000 L CNN
-F 2 "" H 4400 4200 50  0001 C CNN
+F 2 "Connector_JST:JST_PH_B2B-PH-K_1x02_P2.00mm_Vertical" H 4400 4200 50  0001 C CNN
 F 3 "~" H 4400 4200 50  0001 C CNN
 	1    4400 4200
@@
 F 0 "J4" H 4480 4542 50  0000 L CNN
 F 1 "LIMIT_Y" H 4480 4451 50  0000 L CNN
-F 2 "" H 4400 4550 50  0001 C CNN
+F 2 "Connector_JST:JST_PH_B2B-PH-K_1x02_P2.00mm_Vertical" H 4400 4550 50  0001 C CNN
 F 3 "~" H 4400 4550 50  0001 C CNN
 	1    4400 4550
@@
 F 0 "J6" H 7930 2592 50  0000 L CNN
 F 1 "MOTOR_X" H 7930 2501 50  0000 L CNN
-F 2 "" H 7850 2600 50  0001 C CNN
+F 2 "Connector_JST:JST_PH_B4B-PH-K_1x04_P2.00mm_Vertical" H 7850 2600 50  0001 C CNN
 F 3 "~" H 7850 2600 50  0001 C CNN
 	1    7850 2600

Commit message: finish layout and print schematics
Parts:
- removed C3, C7: 100n, Capacitor_SMD:C_0805_2012Metric, symbol Device:C
- removed C6: 10u, Capacitor_SMD:C_0805_2012Metric, symbol Device:CP
- removed TP1, TP2, TP3, TP4, TP5, TP6: TestPoint_2Pole, TestPoint:TestPoint_2Pads_Pitch2.54mm_Drill0.8mm, symbol Connector:TestPoint_2Pole
- added C9: 100u, Capacitor_SMD:CP_Elec_6.3x7.7, symbol Device:CP
- added J8: I2C, Connector_JST:JST_PH_B4B-PH-K_1x04_P2.00mm_Vertical, symbol Connector:Conn_01x04_Female
- C1: footprint Capacitor_SMD:C_0805_2012Metric -> Capacitor_SMD:C_0805_2012Metric_Pad1.15x1.40mm_HandSolder
- R1: footprint Resistor_SMD:R_0805_2012Metric -> Resistor_SMD:R_0805_2012Metric_Pad1.15x1.40mm_HandSolder
- Y1: footprint Crystal:Crystal_SMD_2012-2Pin_2.0x1.2mm -> Crystal:Crystal_SMD_Abracon_ABM3-2Pin_5.0x3.2mm_HandSoldering
Connections:
- net +3V3: now also A1.10 (M0), A1.11 (M1), A1.12 (M2), A2.10 (M0), A2.11 (M1), A2.12 (M2), J8.1 (Pin_1)
- net GND: now also C9.2, J8.4 (Pin_4)
- net at A1.8 (VMOT), A2.8 (VMOT), C8.1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: now also C9.1
- net GPIO2_SDA1 renamed SDA
- net SDA: now also J8.2 (Pin_2)
- net GPIO3_SCL1 renamed SCL
- net SCL: now also J8.3 (Pin_3)
- no-connect marks 38 -> 36
Other:
- note added: "Optional I2C connector"
- moved on the sheet: J1

Commit message: start working on rev1, work in progress
Parts:
- U1: symbol MCU_Microchip_ATmega:ATmega328P-AU -> pizero_grbl_hat-rescue:ATmega328P-AU-MCU_Microchip_ATmega
Changed lines of the file:
@@
 EESchema Schematic File Version 4
-LIBS:pizero_grbl_hat-cache
 EELAYER 30 0
 EELAYER END
@@
 $EndComp
 $Comp
-L MCU_Microchip_ATmega:ATmega328P-AU U1
+L pizero_grbl_hat-rescue:ATmega328P-AU-MCU_Microchip_ATmega U1
 U 1 1 5DD68213
 P 2150 2900
