File: board/pizero_grbl_hat.kicad_pcb (KiCad board)
At the start: 2 copper layers, 65 x 30 mm, 24 parts, among them J1 GPIO_CONNECTOR, J2 ISP, U1 ATmega328P-AU, Y1 16MHz

Commit message: add open hardware logo on the board
Parts:
- added REF**: OSHW-Logo2_9.8x8mm_SilkScreen, Symbol:OSHW-Logo2_9.8x8mm_SilkScreen, F.Cu at (166.8, 106.6)

Commit message: use AVR symbol from the standard library instead of rescue lib
Parts:
- renumbered X-Axis to A1, Y-Axis to A2, Limit-X to J3, Limit-Y to J4, VSTEP to J5, Motor-X to J6, Motor-Y to J7, I2C to J8
Changed lines of the file:
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@@
     (descr "Pololu Breakout 16-pin 15.2x20.3mm 0.6x0.8\\")
     (tags "Pololu Breakout")
-    (fp_text reference X-Axis (at 6.35 -2.032 90) (layer F.SilkS)
+    (fp_text reference A1 (at 6.35 -2.032 90) (layer F.SilkS)
       (effects (font (size 1 1) (thickness 0.15)))
     )
@@
     (descr "Pololu Breakout 16-pin 15.2x20.3mm 0.6x0.8\\")
     (tags "Pololu Breakout")
-    (fp_text reference Y-Axis (at 6.35 -2.54 90) (layer F.SilkS)
+    (fp_text reference A2 (at 6.35 -2.54 90) (layer F.SilkS)
       (effects (font (size 1 1) (thickness 0.15)))
     )
@@
     (descr "JST PH series connector, B4B-PH-K (http://www.jst-mfg.com/product/pdf/eng/ePH.pdf), generated with kicad-footprint-generator")
     (tags "connector JST PH side entry")
-    (fp_text reference Motor-X (at 3 -2.9) (layer F.SilkS)
+    (fp_text reference J6 (at 3 -2.9) (layer F.SilkS)
       (effects (font (size 1 1) (thickness 0.15)))
     )
@@
     (descr "JST PH series connector, B2B-PH-K (http://www.jst-mfg.com/product/pdf/eng/ePH.pdf), generated with kicad-footprint-generator")
     (tags "connector JST PH side entry")
-    (fp_text reference Limit-X (at 1 -2.9) (layer F.SilkS)
+    (fp_text reference J3 (at 1 -2.9) (layer F.SilkS)
       (effects (font (size 1 1) (thickness 0.15)))
     )
@@
     (descr "JST PH series connector, B2B-PH-K (http://www.jst-mfg.com/product/pdf/eng/ePH.pdf), generated with kicad-footprint-generator")
     (tags "connector JST PH side entry")
-    (fp_text reference Limit-Y (at 1 -2.9) (layer F.SilkS)
+    (fp_text reference J4 (at 1 -2.9) (layer F.SilkS)
       (effects (font (size 1 1) (thickness 0.15)))
     )
@@
     (descr "JST PH series connector, B2B-PH-K (http://www.jst-mfg.com/product/pdf/eng/ePH.pdf), generated with kicad-footprint-generator")
     (tags "connector JST PH side entry")
-    (fp_text reference VSTEP (at 1 -2.9) (layer F.SilkS)
+    (fp_text reference J5 (at 1 -2.9) (layer F.SilkS)
       (effects (font (size 1 1) (thickness 0.15)))
     )
@@
     (descr "JST PH series connector, B4B-PH-K (http://www.jst-mfg.com/product/pdf/eng/ePH.pdf), generated with kicad-footprint-generator")
     (tags "connector JST PH side entry")
-    (fp_text reference Motor-Y (at 3 -2.9) (layer F.SilkS)
+    (fp_text reference J7 (at 3 -2.9) (layer F.SilkS)
       (effects (font (size 1 1) (thickness 0.15)))
     )
@@
     (descr "JST PH series connector, B4B-PH-K (http://www.jst-mfg.com/product/pdf/eng/ePH.pdf), generated with kicad-footprint-generator")
     (tags "connector JST PH side entry")
-    (fp_text reference I2C (at 9.3975 1.651 180) (layer F.SilkS)
-      (effects (font (size 1 1) (thickness 0.15)))
-    )
+    (fp_text reference J8 (at 9.3975 1.651 180) (layer F.SilkS)
+      (effects (font (size 1 1) (thickness 0.15)))
+    )
