File: board/pizero_grbl_hat.sch (KiCad schematic (older format))
At the start: 24 parts, among them J1 GPIO_CONNECTOR, J2 ISP, J3 LIMIT_X, J4 LIMIT_Y, J5 VMOT, J6 MOTOR_X, J7 MOTOR_Y, J8 I2C, U1 ATmega328P-AU, Y1 16MHz

Commit message: dome doc updates to schematics
Other:
- note added: "Pololu module is hard-wired\nto 32 micro-steps!"
Changed lines of the file:
@@
 Sheet 1 1
 Title "Raspberry Pi Zero GRBL Hat"
-Date "2019-11-19"
+Date "2020-04-26"
 Rev "1.0"
-Comp "Daniel Winters"
+Comp "Daniel Winters <daniel@tydirium.org>"
 Comment1 "MIT License"
 Comment2 ""
@@
 Wire Wire Line
 	9050 1600 9050 1700
+Text Notes 5600 3500 0    50   ~ 0
+Pololu module is hard-wired\nto 32 micro-steps!
+Text Notes 8050 3500 0    50   ~ 0
+Pololu module is hard-wired\nto 32 micro-steps!
 $EndSCHEMATC

Commit message: use AVR symbol from the standard library instead of rescue lib
Parts:
- U1: symbol pizero_grbl_hat-rescue:ATmega328P-AU-MCU_Microchip_ATmega -> MCU_Microchip_ATmega:ATmega328P-AU
Changed lines of the file:
@@
 $EndComp
 $Comp
-L pizero_grbl_hat-rescue:ATmega328P-AU-MCU_Microchip_ATmega U1
+L MCU_Microchip_ATmega:ATmega328P-AU U1
 U 1 1 5DD68213
 P 2150 2900
